File: kicad/leds.kicad_sch (KiCad schematic)
At the start: 12 parts, among them P1 WJ127-5.0-2P, Q1 IRF7201, Q2 IRF7201, Q3 IRF7201, U1 ESP-F, U3 LM2575HVS-3.3_C347428

Commit message: changed the pcb file to add headers
Parts:
- added J1: Conn_01x04, Connector_PinHeader_2.54mm:PinHeader_1x04_P2.54mm_Vertical, symbol Connector_Generic:Conn_01x04
- C1, C2: footprint Capacitor_THT:CP_Radial_D8.0mm_P3.50mm -> easyeda2kicad:CAP-SMD_BD6.3-L6.6-W6.6-FD
Connections:
- net GND: now also J1.1 (Pin_1)
- net VCC: now reaches C2.1, L1.2, R1.1, U1.3 (EN), U1.8 (VCC), U3.4 (FB)
- net VCC: now also J1.2 (Pin_2)
- net at U1.21 (RXD): now also J1.4 (Pin_4)
- net at U1.22 (TXD): now also J1.3 (Pin_3)
